File: Hardware/LuMini_3Inch.brd (EAGLE design)
At the start: 76.2 x 76.2 mm, 77 parts, among them J1 DOUBLE_LED_PAD, J2 DOUBLE_LED_PAD, J3 DOUBLE_LED_PAD

Commit message: adding silk
Parts:
- added LOGO1: OSHW-LOGOS, SparkFun-Aesthetics:OSHW-LOGO-S
- added LOGO2: SFE_LOGO_NAME.1_INCH, SparkFun-Aesthetics:SFE_LOGO_NAME_.1
- added U$11: (no value), buzzard_labels (5):207
- added U$12: (no value), buzzard_labels (5):258
- added U$13: (no value), buzzard_labels (5):309
- added U$14: (no value), buzzard_labels (5):3510
- added U$15: (no value), buzzard_labels (5):4011
- added U$16: (no value), buzzard_labels (5):5013
- added U$17: (no value), buzzard_labels (5):5514
- added U$3: (no value), buzzard_labels (5):54
- added U$6: (no value), buzzard_labels (5):105
- moved U$1 74.4 mm to (34.9, 1.08), turned to 180 degrees
- moved U$2 69.6 mm to (31.6, 4.00), turned to 180 degrees
Routing:
- net N$42: track 0.00 -> 2.02 mm
- net N$60: track 0.00 -> 1.93 mm
Changed lines of the file:
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@@
 <setting verticaltext="up"/>
 </settings>
-<grid distance="0.05" unitdist="inch" unit="inch" style="lines" multiple="1" display="yes" altdistance="0.005" altunitdist="inch" altunit="inch"/>
+<grid distance="0.05" unitdist="inch" unit="inch" style="lines" multiple="1" display="yes" altdistance="0.0005" altunitdist="inch" altunit="inch"/>
 <layers>
 <layer number="1" name="Top" color="4" fill="1" visible="yes" active="yes"/>
@@
 <layer number="19" name="Unrouted" color="6" fill="1" visible="yes" active="yes"/>
 <layer number="20" name="Dimension" color="24" fill="1" visible="yes" active="yes"/>
-<layer number="21" name="tPlace" color="7" fill="1" visible="yes" active="yes"/>
+<layer number="21" name="tPlace" color="16" fill="1" visible="yes" active="yes"/>
 <layer number="22" name="bPlace" color="7" fill="1" visible="yes" active="yes"/>
 <layer number="23" name="tOrigins" color="15" fill="1" visible="yes" active="yes"/>
@@
 <element name="J1" library="Andy" package="DOUBLELEDPAD" value="DOUBLE_LED_PAD" x="73.8505" y="41.3385" rot="MR266.4"/>
 <element name="J2" library="Andy" package="DOUBLELEDPAD" value="DOUBLE_LED_PAD" x="73.9775" y="37.4142" rot="MR270"/>
-<element name="U$1" library="buzzard_labels (2)" package="LUMINI0" value="" x="41.275" y="75.2475" rot="MR0"/>
+<element name="U$1" library="buzzard_labels (2)" package="LUMINI0" value="" x="34.925" y="1.0795" rot="MR180"/>
 <element name="U$4" library="buzzard_labels (25)" package="5V6" value="" x="71.6915" y="41.529" rot="MR266.4"/>
 <element name="U$5" library="buzzard_labels (25)" package="G4" value="" x="71.501" y="43.307" rot="MR266.4"/>
@@
 </element>
 <element name="J3" library="Andy" package="DOUBLELEDPAD" value="DOUBLE_LED_PAD" x="73.6727" y="33.2994" rot="MR97"/>
-<element name="U$2" library="buzzard_labels (3)" package="60_APA102_LEDS0" value="" x="44.6405" y="72.3265" rot="MR0"/>
+<element name="U$2" library="buzzard_labels (3)" package="60_APA102_LEDS0" value="" x="31.5595" y="4.0005" rot="MR180"/>
 <element name="FRAME1" library="SparkFun-Aesthetics" package="CREATIVE_COMMONS" value="FRAME-LEDGER" x="14.605" y="-8.255">
 <attribute name="DESIGNER" value="" x="14.605" y="-8.255" size="1.778" layer="27" display="off"/>
@@
 <attribute name="PROD_ID" value="CAP-08280" x="69.977" y="26.797" size="1.778" layer="28" rot="MR110" display="off"/>
 </element>
+<element name="LOGO1" library="SparkFun-Aesthetics" package="OSHW-LOGO-S" value="OSHW-LOGOS" x="2.921" y="34.417" rot="MR264"/>
+<element name="LOGO2" library="SparkFun-Aesthetics" package="SFE_LOGO_NAME_.1" value="SFE_LOGO_NAME.1_INCH" x="38.1" y="72.39" rot="MR0"/>
+<element name="U$3" library="buzzard_labels (5)" package="54" value="" x="69.469" y="54.483" rot="MR60"/>
+<element name="U$6" library="buzzard_labels (5)" package="105" value="" x="57.1881" y="67.9577" rot="MR30"/>
+<element name="U$11" library="buzzard_labels (5)" package="207" value="" x="21.9202" y="69.6468" rot="MR330"/>
+<element name="U$12" library="buzzard_labels (5)" package="258" value="" x="8.2931" y="57.3024" rot="MR300"/>
+<element name="U$13" library="buzzard_labels (5)" package="309" value="" x="2.5019" y="36.3347" rot="MR90"/>
+<element name="U$14" library="buzzard_labels (5)" package="3510" value="" x="6.5532" y="21.844" rot="MR240"/>
+<element name="U$15" library="buzzard_labels (5)" package="4011" value="" x="18.8595" y="8.3439" rot="MR210"/>
+<element name="U$16" library="buzzard_labels (5)" package="5013" value="" x="54.1528" y="6.4897" rot="MR150"/>
+<element name="U$17" library="buzzard_labels (5)" package="5514" value="" x="67.9704" y="18.9611" rot="MR120"/>
 </elements>
 <signals>
@@
 <contactref element="D16" pad="CKI"/>
 <contactref element="D15" pad="CKO"/>
-<wire x1="38.94491875" y1="73.535540625" x2="40.960515625" y2="73.431346875" width="0" layer="19" extent="1-1"/>
+<wire x1="40.960515625" y1="73.431346875" x2="38.94491875" y2="73.535540625" width="0.1778" layer="1"/>
 </signal>
 <signal name="N$60">
 <contactref element="D15" pad="SDO"/>
 <contactref element="D16" pad="SDI"/>
-<wire x1="38.94491875" y1="72.735540625" x2="40.876890625" y2="72.63573125" width="0" layer="19" extent="1-1"/>
+<wire x1="38.94491875" y1="72.735540625" x2="40.876890625" y2="72.63573125" width="0.1778" layer="1"/>
 </signal>
 <signal name="N$61">

Commit message: post checklist
Parts:
- added FD1, FD2, FD3, FD4: FIDUCIALUFIDUCIAL, SparkFun-Aesthetics:FIDUCIAL-MICRO
- added H5, H6, H7, H8: STANDOFF_ELECTRICALSTANDOFF-ELECTRICAL-NOTHERMALS, SparkFun-Hardware:STANDOFF-ELECTRICAL-NOTHERMALS
- added U$18: (no value), SparkFun-Aesthetics:ORDERING_INSTRUCTIONS
- C1: value 4.7uF -> DNP; device SparkFun-Capacitors:0603 -> SparkFun-Capacitors:1206
- U$1: device buzzard_labels (2):LUMINI0 -> buzzard_labels (8):LUMINI_3#2
- moved H2 1.27 mm to (38.1, 8.89)
- moved H4 1.27 mm to (8.89, 38.1)
- moved H1 1.27 mm to (67.3, 38.1)
- moved H3 1.27 mm to (38.1, 67.3)
- moved U$1 0.89 mm to (34.0, 1.08)
- moved C1 0.36 mm to (70.3, 26.6)
Connections:
- net GND: now also H5.P1, H6.P1, H7.P1, H8.P1
Other:
- outline, holes or cut-outs redrawn
- board text added: "Black PCB 2 Oz. Cu"

Commit message: cleaning up schematic
Parts:
- H1, H2, H3, H4, H5, H6, H7, H8: value STANDOFF_ELECTRICALSTANDOFF-ELECTRICAL-NOTHERMALS -> STANDOFF_ELECTRICAL-NOTHERMALS
Connections:
- net N$122 renamed CO
- net N$123 renamed DO
- net N$2 renamed CI
- net N$3 renamed DI
Changed lines of the file:
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@@
 <attribute name="REV" value="" x="14.605" y="-8.255" size="1.778" layer="27" display="off"/>
 </element>
-<element name="H1" library="SparkFun-Hardware" package="STANDOFF-ELECTRICAL-NOTHERMALS" value="STANDOFF_ELECTRICALSTANDOFF-ELECTRICAL-NOTHERMALS" x="67.31" y="38.1"/>
-<element name="H2" library="SparkFun-Hardware" package="STANDOFF-ELECTRICAL-NOTHERMALS" value="STANDOFF_ELECTRICALSTANDOFF-ELECTRICAL-NOTHERMALS" x="38.1" y="8.89"/>
-<element name="H3" library="SparkFun-Hardware" package="STANDOFF-ELECTRICAL-NOTHERMALS" value="STANDOFF_ELECTRICALSTANDOFF-ELECTRICAL-NOTHERMALS" x="38.1" y="67.31"/>
-<element name="H4" library="SparkFun-Hardware" package="STANDOFF-ELECTRICAL-NOTHERMALS" value="STANDOFF_ELECTRICALSTANDOFF-ELECTRICAL-NOTHERMALS" x="8.89" y="38.1"/>
+<element name="H1" library="SparkFun-Hardware" package="STANDOFF-ELECTRICAL-NOTHERMALS" value="STANDOFF_ELECTRICAL-NOTHERMALS" x="67.31" y="38.1"/>
+<element name="H2" library="SparkFun-Hardware" package="STANDOFF-ELECTRICAL-NOTHERMALS" value="STANDOFF_ELECTRICAL-NOTHERMALS" x="38.1" y="8.89"/>
+<element name="H3" library="SparkFun-Hardware" package="STANDOFF-ELECTRICAL-NOTHERMALS" value="STANDOFF_ELECTRICAL-NOTHERMALS" x="38.1" y="67.31"/>
+<element name="H4" library="SparkFun-Hardware" package="STANDOFF-ELECTRICAL-NOTHERMALS" value="STANDOFF_ELECTRICAL-NOTHERMALS" x="8.89" y="38.1"/>
 <element name="C1" library="SparkFun-Capacitors" package="1206" value="DNP" x="70.2945" y="26.6319" rot="MR110">
 <attribute name="PROD_ID" value="CAP-10300" x="70.2945" y="26.6319" size="1.778" layer="28" rot="MR110" display="off"/>
@@
 <element name="U$16" library="buzzard_labels (5)" package="5013" value="" x="54.1528" y="6.4897" rot="MR150"/>
 <element name="U$17" library="buzzard_labels (5)" package="5514" value="" x="67.9704" y="18.9611" rot="MR120"/>
-<element name="H5" library="SparkFun-Hardware" package="STANDOFF-ELECTRICAL-NOTHERMALS" value="STANDOFF_ELECTRICALSTANDOFF-ELECTRICAL-NOTHERMALS" x="8.89" y="8.89"/>
-<element name="H6" library="SparkFun-Hardware" package="STANDOFF-ELECTRICAL-NOTHERMALS" value="STANDOFF_ELECTRICALSTANDOFF-ELECTRICAL-NOTHERMALS" x="67.31" y="8.89"/>
-<element name="H7" library="SparkFun-Hardware" package="STANDOFF-ELECTRICAL-NOTHERMALS" value="STANDOFF_ELECTRICALSTANDOFF-ELECTRICAL-NOTHERMALS" x="8.89" y="67.31"/>
-<element name="H8" library="SparkFun-Hardware" package="STANDOFF-ELECTRICAL-NOTHERMALS" value="STANDOFF_ELECTRICALSTANDOFF-ELECTRICAL-NOTHERMALS" x="67.31" y="67.31"/>
+<element name="H5" library="SparkFun-Hardware" package="STANDOFF-ELECTRICAL-NOTHERMALS" value="STANDOFF_ELECTRICAL-NOTHERMALS" x="8.89" y="8.89"/>
+<element name="H6" library="SparkFun-Hardware" package="STANDOFF-ELECTRICAL-NOTHERMALS" value="STANDOFF_ELECTRICAL-NOTHERMALS" x="67.31" y="8.89"/>
+<element name="H7" library="SparkFun-Hardware" package="STANDOFF-ELECTRICAL-NOTHERMALS" value="STANDOFF_ELECTRICAL-NOTHERMALS" x="8.89" y="67.31"/>
+<element name="H8" library="SparkFun-Hardware" package="STANDOFF-ELECTRICAL-NOTHERMALS" value="STANDOFF_ELECTRICAL-NOTHERMALS" x="67.31" y="67.31"/>
 <element name="FD1" library="SparkFun-Aesthetics" package="FIDUCIAL-MICRO" value="FIDUCIALUFIDUCIAL" x="8.382" y="12.573"/>
 <element name="FD2" library="SparkFun-Aesthetics" package="FIDUCIAL-MICRO" value="FIDUCIALUFIDUCIAL" x="8.382" y="12.573" rot="MR90"/>
@@
 <wire x1="74.041" y1="30.4165" x2="73.72008125" y2="31.401634375" width="0.2032" layer="1"/>
 </signal>
-<signal name="N$2">
+<signal name="CI">
 <contactref element="D1" pad="CKI"/>
 <contactref element="J2" pad="P$2"/>
@@
 <wire x1="73.9775" y1="36.3982" x2="73.914" y2="36.3347" width="0.1778" layer="16"/>
 </signal>
-<signal name="N$3">
+<signal name="DI">
 <contactref element="D1" pad="SDI"/>
 <contactref element="J2" pad="P$1"/>
@@
 <wire x1="69.2082" y1="21.117078125" x2="70.121490625" y2="22.914065625" width="0.1778" layer="1"/>
 </signal>
-<signal name="N$122">
+<signal name="CO">
 <contactref element="D60" pad="CKO"/>
 <contactref element="J3" pad="P$2"/>
@@
 <wire x1="73.3425" y1="34.671" x2="73.66" y2="34.29" width="0.1778" layer="1"/>
 </signal>
-<signal name="N$123">
+<signal name="DO">
 <contactref element="D60" pad="SDO"/>
 <contactref element="J3" pad="P$1"/>

Commit message: fixing library issue
Parts:
- J1, J2, J3: value DOUBLE_LED_PAD -> SOLDER_PAD_2; device Andy:DOUBLELEDPAD -> SparkFun-Connectors:SOLDER_PAD_2
Changed lines of the file:
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@@
 <attribute name="PROD_ID" value="DIO-13883" x="37.41715" y="64.91578125" size="1.778" layer="27" rot="R204" display="off"/>
 </element>
-<element name="J1" library="Andy" package="DOUBLELEDPAD" value="DOUBLE_LED_PAD" x="73.8505" y="41.3385" rot="MR266.4"/>
-<element name="J2" library="Andy" package="DOUBLELEDPAD" value="DOUBLE_LED_PAD" x="73.9775" y="37.4142" rot="MR270"/>
+<element name="J1" library="SparkFun-Connectors" package="SOLDER_PAD_2" value="SOLDER_PAD_2" x="73.8505" y="41.3385" rot="MR266.4"/>
+<element name="J2" library="SparkFun-Connectors" package="SOLDER_PAD_2" value="SOLDER_PAD_2" x="73.9775" y="37.4142" rot="MR270"/>
 <element name="U$1" library="buzzard_labels (8)" package="LUMINI_3#2" value="" x="34.036" y="1.0795" rot="MR180"/>
 <element name="U$4" library="buzzard_labels (25)" package="5V6" value="" x="71.6915" y="41.529" rot="MR266.4"/>
@@
 <attribute name="PROD_ID" value="DIO-13883" x="35.38531875" y="-72.599775" size="1.778" layer="27" rot="R84" display="off"/>
 </element>
-<element name="J3" library="Andy" package="DOUBLELEDPAD" value="DOUBLE_LED_PAD" x="73.6727" y="33.2994" rot="MR97"/>
+<element name="J3" library="SparkFun-Connectors" package="SOLDER_PAD_2" value="SOLDER_PAD_2" x="73.6727" y="33.2994" rot="MR97"/>
 <element name="U$2" library="buzzard_labels (3)" package="60_APA102_LEDS0" value="" x="31.5595" y="4.0005" rot="MR180"/>
 <element name="FRAME1" library="SparkFun-Aesthetics" package="CREATIVE_COMMONS" value="FRAME-LEDGER" x="14.605" y="-8.255">

Commit message: updating to proper 6-pin footprint
Parts:
- D1, D10, D11, D12, D13, D14, D15, D16, D17, D18, D19, D2, D20, D21, D22, D23, D24, D25, D26, D27, D28, D29, D3, D30, D31, D32, D33, D34, D35, D36, D37, D38, D39, D4, D40, D41, D42, D43, D44, D45, D46, D47, D48, D49, D5, D50, D51, D52, D53, D54, D55, D56, D57, D58, D59, D6, D60, D7, D8, D9: value APA1022020 -> APA102-2020
- moved U$13 3.53 mm to (2.58, 39.9), turned to 270 degrees
- moved U$7 3.19 mm to (71.4, 31.0), turned to 97 degrees
- moved U$8 3.07 mm to (71.6, 33.1), turned to 97 degrees
- moved U$4 2.80 mm to (71.8, 38.7), turned to 86.4 degrees
- moved U$9 2.62 mm to (71.9, 35.1), turned to 90 degrees
- moved U$10 2.54 mm to (71.8, 37.1), turned to 90 degrees
- moved U$5 2.29 mm to (71.6, 41.0), turned to 86.4 degrees
Routing:
- net 5V: track 62.6 -> 4.53 mm, vias 60 -> 2
- net GND: track 1.96 -> 2.86 mm, vias 2 -> 5
- net DI: track 3.55 -> 4.11 mm
- added copper zone on layer 1, net 5V
- added copper zone on layer 16, net GND
- removed copper zone on layer 16, net 5V

Commit message: version number change
Other:
- board text added: "v10"
- board text removed: "v03"
Changed lines of the file:
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@@
 <plain>
 <circle x="38.1" y="38.1" radius="38.1" width="0.2032" layer="21"/>
-<text x="5.08" y="40.005" size="1.778" layer="16" font="vector" ratio="15" rot="SMR270">v03</text>
+<text x="5.08" y="40.005" size="1.778" layer="16" font="vector" ratio="15" rot="SMR270">v10</text>
 <text x="41.402" y="-8.3185" size="1.778" layer="51" font="vector">Andy England</text>
 <wire x1="5.588" y1="41.91" x2="8.89" y2="41.91" width="0.2032" layer="20"/>
