File: Hardware/LuMini_3Inch.brd (EAGLE design)
At the start: 166.6 x 243.3 mm, 573 parts, among them J1 SOLDER_PAD_2, J10 SOLDER_PAD_2, J11 SOLDER_PAD_2, J12 SOLDER_PAD_2, J13 SOLDER_PAD_2, J14 SOLDER_PAD_2, J15 SOLDER_PAD_2, J16 SOLDER_PAD_2, J17 SOLDER_PAD_2, J18 SOLDER_PAD_2, J2 SOLDER_PAD_2, J3 SOLDER_PAD_2, J4 SOLDER_PAD_2, J5 SOLDER_PAD_2, J6 SOLDER_PAD_2, J7 SOLDER_PAD_2, J8 SOLDER_PAD_2, J9 SOLDER_PAD_2

Commit message: production saved over the original design with a panel. Changed back to the original design
Parts:
- removed C2, C3, C4, C5, C6: DNP, SparkFun-Capacitors:1206
- removed D100, D101, D102, D103, D104, D105, D106, D107, D108, D109, D110, D111, D112, D113, D114, D115, D116, D117, D118, D119, D120, D121, D122, D123, D124, D125, D126, D127, D128, D129, D130, D131, D132, D133, D134, D135, D136, D137, D138, D139, D140, D141, D142, D143, D144, D145, D146, D147, D148, D149, D150, D151, D152, D153, D154, D155, D156, D157, D158, D159, D160, D161, D162, D163, D164, D165, D166, D167, D168, D169, D170, D171, D172, D173, D174, D175, D176, D177, D178, D179, D180, D181, D182, D183, D184, D185, D186, D187, D188, D189, D190, D191, D192, D193, D194, D195, D196, D197, D198, D199, D200, D201, D202, D203, D204, D205, D206, D207, D208, D209, D210, D211, D212, D213, D214, D215, D216, D217, D218, D219, D220, D221, D222, D223, D224, D225, D226, D227, D228, D229, D230, D231, D232, D233, D234, D235, D236, D237, D238, D239, D240, D241, D242, D243, D244, D245, D246, D247, D248, D249, D250, D251, D252, D253, D254, D255, D256, D257, D258, D259, D260, D261, D262, D263, D264, D265, D266, D267, D268, D269, D270, D271, D272, D273, D274, D275, D276, D277, D278, D279, D280, D281, D282, D283, D284, D285, D286, D287, D288, D289, D290, D291, D292, D293, D294, D295, D296, D297, D298, D299, D300, D301, D302, D303, D304, D305, D306, D307, D308, D309, D310, D311, D312, D313, D314, D315, D316, D317, D318, D319, D320, D321, D322, D323, D324, D325, D326, D327, D328, D329, D330, D331, D332, D333, D334, D335, D336, D337, D338, D339, D340, D341, D342, D343, D344, D345, D346, D347, D348, D349, D350, D351, D352, D353, D354, D355, D356, D357, D358, D359, D360, D61, D62, D63, D64, D65, D66, D67, D68, D69, D70, D71, D72, D73, D74, D75, D76, D77, D78, D79, D80, D81, D82, D83, D84, D85, D86, D87, D88, D89, D90, D91, D92, D93, D94, D95, D96, D97, D98, D99: APA102-2020, SparkFun-LED:APA102-2020
- removed E$6: (no value), SparkFun-Retired:FIDUCIAL-1.5X3
- removed E$7, E$8: (no value), SparkFun-Aesthetics:FIDUCIAL-1X2
- removed FD10, FD11, FD12, FD13, FD14, FD15, FD16, FD17, FD18, FD19, FD20, FD21, FD22, FD23, FD24, FD5, FD6, FD7, FD8, FD9: FIDUCIALUFIDUCIAL, SparkFun-Aesthetics:FIDUCIAL-MICRO
- removed H10, H11, H12, H13, H14, H15, H16, H17, H18, H19, H20, H21, H22, H23, H24, H25, H26, H27, H28, H29, H30, H31, H32, H33, H34, H35, H36, H37, H38, H39, H40, H41, H42, H43, H44, H45, H46, H47, H48, H9: STANDOFF_ELECTRICAL-NOTHERMALS, SparkFun-Hardware:STANDOFF-ELECTRICAL-NOTHERMALS
- removed J10, J11, J12, J13, J14, J15, J16, J17, J18, J4, J5, J6, J7, J8, J9: SOLDER_PAD_2, SparkFun-Connectors:SOLDER_PAD_2
- removed LOGO10, LOGO12, LOGO4, LOGO6, LOGO8: SFE_LOGO_NAME.1_INCH, SparkFun-Aesthetics:SFE_LOGO_NAME_.1
- removed LOGO11, LOGO3, LOGO5, LOGO7, LOGO9: OSHW-LOGOS, SparkFun-Aesthetics:OSHW-LOGO-S
- removed U$100, U$32, U$49, U$66, U$83: (no value), buzzard_labels (5):4011
- removed U$101, U$33, U$50, U$67, U$84: (no value), buzzard_labels (5):5013
- removed U$102, U$34, U$51, U$68, U$85: (no value), buzzard_labels (5):5514
- removed U$19, U$36, U$53, U$70, U$87: (no value), buzzard_labels (25):5V6
- removed U$20, U$37, U$54, U$71, U$88: (no value), buzzard_labels (25):G4
- removed U$21, U$38, U$55, U$72, U$89: (no value), buzzard_labels (25):DO3
- removed U$22, U$39, U$56, U$73, U$90: (no value), buzzard_labels (25):CO1
- removed U$23, U$40, U$57, U$74, U$91: (no value), buzzard_labels (26):CI6
- removed U$24, U$41, U$58, U$75, U$92: (no value), buzzard_labels (26):DI4
- removed U$25, U$42, U$59, U$76, U$93: (no value), buzzard_labels (3):60_APA102_LEDS0
- removed U$26, U$43, U$60, U$77, U$94: (no value), buzzard_labels (5):54
- removed U$27, U$44, U$61, U$78, U$95: (no value), buzzard_labels (5):105
- removed U$28, U$45, U$62, U$79, U$96: (no value), buzzard_labels (5):207
- removed U$29, U$46, U$63, U$80, U$97: (no value), buzzard_labels (5):258
- removed U$30, U$47, U$64, U$81, U$98: (no value), buzzard_labels (5):309
- removed U$31, U$48, U$65, U$82, U$99: (no value), buzzard_labels (5):3510
- removed U$35, U$52, U$69, U$86: (no value), buzzard_labels (8):LUMINI_3#2
- added FRAME1: FRAME-LEDGER, SparkFun-Aesthetics:CREATIVE_COMMONS
- U$18: device buzzard_labels (8):LUMINI_3#2 -> SparkFun-Aesthetics:ORDERING_INSTRUCTIONS
- moved U$18 121.0 mm to (-9.65, -11.2), flipped to the top, turned to 0 degrees
Connections:
- removed net 5V1: C2.1, D100.VDD, D101.VDD, D102.VDD, D103.VDD, D104.VDD, D105.VDD, D106.VDD, D107.VDD, D108.VDD, D109.VDD, D110.VDD, D111.VDD, D112.VDD, D113.VDD, D114.VDD, D115.VDD, D116.VDD, D117.VDD, D118.VDD, D119.VDD, D120.VDD, D61.VDD, D62.VDD, D63.VDD, D64.VDD, D65.VDD, D66.VDD, D67.VDD, D68.VDD, D69.VDD, D70.VDD, D71.VDD, D72.VDD, D73.VDD, D74.VDD, D75.VDD, D76.VDD, D77.VDD, D78.VDD, D79.VDD, D80.VDD, D81.VDD, D82.VDD, D83.VDD, D84.VDD, D85.VDD, D86.VDD, D87.VDD, D88.VDD, D89.VDD, D90.VDD, D91.VDD, D92.VDD, D93.VDD, D94.VDD, D95.VDD, D96.VDD, D97.VDD, D98.VDD, D99.VDD, J4.P$2
- removed net 5V2: C3.1, D121.VDD, D122.VDD, D123.VDD, D124.VDD, D125.VDD, D126.VDD, D127.VDD, D128.VDD, D129.VDD, D130.VDD, D131.VDD, D132.VDD, D133.VDD, D134.VDD, D135.VDD, D136.VDD, D137.VDD, D138.VDD, D139.VDD, D140.VDD, D141.VDD, D142.VDD, D143.VDD, D144.VDD, D145.VDD, D146.VDD, D147.VDD, D148.VDD, D149.VDD, D150.VDD, D151.VDD, D152.VDD, D153.VDD, D154.VDD, D155.VDD, D156.VDD, D157.VDD, D158.VDD, D159.VDD, D160.VDD, D161.VDD, D162.VDD, D163.VDD, D164.VDD, D165.VDD, D166.VDD, D167.VDD, D168.VDD, D169.VDD, D170.VDD, D171.VDD, D172.VDD, D173.VDD, D174.VDD, D175.VDD, D176.VDD, D177.VDD, D178.VDD, D179.VDD, D180.VDD, J7.P$2
- removed net 5V3: C4.1, D181.VDD, D182.VDD, D183.VDD, D184.VDD, D185.VDD, D186.VDD, D187.VDD, D188.VDD, D189.VDD, D190.VDD, D191.VDD, D192.VDD, D193.VDD, D194.VDD, D195.VDD, D196.VDD, D197.VDD, D198.VDD, D199.VDD, D200.VDD, D201.VDD, D202.VDD, D203.VDD, D204.VDD, D205.VDD, D206.VDD, D207.VDD, D208.VDD, D209.VDD, D210.VDD, D211.VDD, D212.VDD, D213.VDD, D214.VDD, D215.VDD, D216.VDD, D217.VDD, D218.VDD, D219.VDD, D220.VDD, D221.VDD, D222.VDD, D223.VDD, D224.VDD, D225.VDD, D226.VDD, D227.VDD, D228.VDD, D229.VDD, D230.VDD, D231.VDD, D232.VDD, D233.VDD, D234.VDD, D235.VDD, D236.VDD, D237.VDD, D238.VDD, D239.VDD, D240.VDD, J10.P$2
- removed net 5V4: C5.1, D241.VDD, D242.VDD, D243.VDD, D244.VDD, D245.VDD, D246.VDD, D247.VDD, D248.VDD, D249.VDD, D250.VDD, D251.VDD, D252.VDD, D253.VDD, D254.VDD, D255.VDD, D256.VDD, D257.VDD, D258.VDD, D259.VDD, D260.VDD, D261.VDD, D262.VDD, D263.VDD, D264.VDD, D265.VDD, D266.VDD, D267.VDD, D268.VDD, D269.VDD, D270.VDD, D271.VDD, D272.VDD, D273.VDD, D274.VDD, D275.VDD, D276.VDD, D277.VDD, D278.VDD, D279.VDD, D280.VDD, D281.VDD, D282.VDD, D283.VDD, D284.VDD, D285.VDD, D286.VDD, D287.VDD, D288.VDD, D289.VDD, D290.VDD, D291.VDD, D292.VDD, D293.VDD, D294.VDD, D295.VDD, D296.VDD, D297.VDD, D298.VDD, D299.VDD, D300.VDD, J13.P$2
- removed net 5V5: C6.1, D301.VDD, D302.VDD, D303.VDD, D304.VDD, D305.VDD, D306.VDD, D307.VDD, D308.VDD, D309.VDD, D310.VDD, D311.VDD, D312.VDD, D313.VDD, D314.VDD, D315.VDD, D316.VDD, D317.VDD, D318.VDD, D319.VDD, D320.VDD, D321.VDD, D322.VDD, D323.VDD, D324.VDD, D325.VDD, D326.VDD, D327.VDD, D328.VDD, D329.VDD, D330.VDD, D331.VDD, D332.VDD, D333.VDD, D334.VDD, D335.VDD, D336.VDD, D337.VDD, D338.VDD, D339.VDD, D340.VDD, D341.VDD, D342.VDD, D343.VDD, D344.VDD, D345.VDD, D346.VDD, D347.VDD, D348.VDD, D349.VDD, D350.VDD, D351.VDD, D352.VDD, D353.VDD, D354.VDD, D355.VDD, D356.VDD, D357.VDD, D358.VDD, D359.VDD, D360.VDD, J16.P$2
- removed net CI1: D61.CKI, J5.P$2
- removed net CI2: D121.CKI, J8.P$2
- removed net CI3: D181.CKI, J11.P$2
- removed net CI4: D241.CKI, J14.P$2
- removed net CI5: D301.CKI, J17.P$2
- removed net CO1: D120.CKO, J6.P$2
- removed net CO2: D180.CKO, J9.P$2
- removed net CO3: D240.CKO, J12.P$2
- removed net CO4: D300.CKO, J15.P$2
- removed net CO5: D360.CKO, J18.P$2
- removed net DI1: D61.SDI, J5.P$1
- removed net DI2: D121.SDI, J8.P$1
- removed net DI3: D181.SDI, J11.P$1
- removed net DI4: D241.SDI, J14.P$1
- removed net DI5: D301.SDI, J17.P$1
- removed net DO1: D120.SDO, J6.P$1
- removed net DO2: D180.SDO, J9.P$1
- removed net DO3: D240.SDO, J12.P$1
- removed net DO4: D300.SDO, J15.P$1
- removed net DO5: D360.SDO, J18.P$1
- removed net GND1: C2.2, D100.GND, D101.GND, D102.GND, D103.GND, D104.GND, D105.GND, D106.GND, D107.GND, D108.GND, D109.GND, D110.GND, D111.GND, D112.GND, D113.GND, D114.GND, D115.GND, D116.GND, D117.GND, D118.GND, D119.GND, D120.GND, D61.GND, D62.GND, D63.GND, D64.GND, D65.GND, D66.GND, D67.GND, D68.GND, D69.GND, D70.GND, D71.GND, D72.GND, D73.GND, D74.GND, D75.GND, D76.GND, D77.GND, D78.GND, D79.GND, D80.GND, D81.GND, D82.GND, D83.GND, D84.GND, D85.GND, D86.GND, D87.GND, D88.GND, D89.GND, D90.GND, D91.GND, D92.GND, D93.GND, D94.GND, D95.GND, D96.GND, D97.GND, D98.GND, D99.GND, H10.P1, H11.P1, H12.P1, H13.P1, H14.P1, H15.P1, H16.P1, H9.P1, J4.P$1
- removed net GND2: C3.2, D121.GND, D122.GND, D123.GND, D124.GND, D125.GND, D126.GND, D127.GND, D128.GND, D129.GND, D130.GND, D131.GND, D132.GND, D133.GND, D134.GND, D135.GND, D136.GND, D137.GND, D138.GND, D139.GND, D140.GND, D141.GND, D142.GND, D143.GND, D144.GND, D145.GND, D146.GND, D147.GND, D148.GND, D149.GND, D150.GND, D151.GND, D152.GND, D153.GND, D154.GND, D155.GND, D156.GND, D157.GND, D158.GND, D159.GND, D160.GND, D161.GND, D162.GND, D163.GND, D164.GND, D165.GND, D166.GND, D167.GND, D168.GND, D169.GND, D170.GND, D171.GND, D172.GND, D173.GND, D174.GND, D175.GND, D176.GND, D177.GND, D178.GND, D179.GND, D180.GND, H17.P1, H18.P1, H19.P1, H20.P1, H21.P1, H22.P1, H23.P1, H24.P1, J7.P$1
- removed net GND3: C4.2, D181.GND, D182.GND, D183.GND, D184.GND, D185.GND, D186.GND, D187.GND, D188.GND, D189.GND, D190.GND, D191.GND, D192.GND, D193.GND, D194.GND, D195.GND, D196.GND, D197.GND, D198.GND, D199.GND, D200.GND, D201.GND, D202.GND, D203.GND, D204.GND, D205.GND, D206.GND, D207.GND, D208.GND, D209.GND, D210.GND, D211.GND, D212.GND, D213.GND, D214.GND, D215.GND, D216.GND, D217.GND, D218.GND, D219.GND, D220.GND, D221.GND, D222.GND, D223.GND, D224.GND, D225.GND, D226.GND, D227.GND, D228.GND, D229.GND, D230.GND, D231.GND, D232.GND, D233.GND, D234.GND, D235.GND, D236.GND, D237.GND, D238.GND, D239.GND, D240.GND, H25.P1, H26.P1, H27.P1, H28.P1, H29.P1, H30.P1, H31.P1, H32.P1, J10.P$1
- removed net GND4: C5.2, D241.GND, D242.GND, D243.GND, D244.GND, D245.GND, D246.GND, D247.GND, D248.GND, D249.GND, D250.GND, D251.GND, D252.GND, D253.GND, D254.GND, D255.GND, D256.GND, D257.GND, D258.GND, D259.GND, D260.GND, D261.GND, D262.GND, D263.GND, D264.GND, D265.GND, D266.GND, D267.GND, D268.GND, D269.GND, D270.GND, D271.GND, D272.GND, D273.GND, D274.GND, D275.GND, D276.GND, D277.GND, D278.GND, D279.GND, D280.GND, D281.GND, D282.GND, D283.GND, D284.GND, D285.GND, D286.GND, D287.GND, D288.GND, D289.GND, D290.GND, D291.GND, D292.GND, D293.GND, D294.GND, D295.GND, D296.GND, D297.GND, D298.GND, D299.GND, D300.GND, H33.P1, H34.P1, H35.P1, H36.P1, H37.P1, H38.P1, H39.P1, H40.P1, J13.P$1
- removed net GND5: C6.2, D301.GND, D302.GND, D303.GND, D304.GND, D305.GND, D306.GND, D307.GND, D308.GND, D309.GND, D310.GND, D311.GND, D312.GND, D313.GND, D314.GND, D315.GND, D316.GND, D317.GND, D318.GND, D319.GND, D320.GND, D321.GND, D322.GND, D323.GND, D324.GND, D325.GND, D326.GND, D327.GND, D328.GND, D329.GND, D330.GND, D331.GND, D332.GND, D333.GND, D334.GND, D335.GND, D336.GND, D337.GND, D338.GND, D339.GND, D340.GND, D341.GND, D342.GND, D343.GND, D344.GND, D345.GND, D346.GND, D347.GND, D348.GND, D349.GND, D350.GND, D351.GND, D352.GND, D353.GND, D354.GND, D355.GND, D356.GND, D357.GND, D358.GND, D359.GND, D360.GND, H41.P1, H42.P1, H43.P1, H44.P1, H45.P1, H46.P1, H47.P1, H48.P1, J16.P$1
- removed net N$122: D72.CKO, D73.CKI
- removed net N$123: D72.SDO, D73.SDI
- removed net N$125: D73.CKO, D74.CKI
- removed net N$126: D73.SDO, D74.SDI
- removed net N$127: D74.CKO, D75.CKI
- removed net N$128: D74.SDO, D75.SDI
- removed net N$129: D75.CKO, D76.CKI
- removed net N$130: D75.SDO, D76.SDI
- removed net N$131: D76.CKO, D77.CKI
- removed net N$132: D76.SDO, D77.SDI
- removed net N$133: D62.CKI, D78.CKO
- removed net N$134: D62.SDI, D78.SDO
- removed net N$135: D62.CKO, D63.CKI
- removed net N$136: D62.SDO, D63.SDI
- removed net N$137: D63.CKO, D64.CKI
- removed net N$138: D63.SDO, D64.SDI
- removed net N$139: D64.CKO, D65.CKI
- removed net N$140: D64.SDO, D65.SDI
- removed net N$141: D65.CKO, D66.CKI
- removed net N$142: D65.SDO, D66.SDI
- removed net N$143: D66.CKO, D67.CKI
- removed net N$144: D66.SDO, D67.SDI
- removed net N$145: D69.CKO, D70.CKI
- removed net N$146: D69.SDO, D70.SDI
- removed net N$147: D70.SDO, D79.SDI
- removed net N$148: D79.CKO, D80.CKI
- removed net N$149: D79.SDO, D80.SDI
- removed net N$150: D70.CKO, D79.CKI
- removed net N$151: D77.CKO, D78.CKI
- removed net N$152: D77.SDO, D78.SDI
- removed net N$153: D68.SDO, D69.SDI
- removed net N$154: D68.CKO, D69.CKI
- removed net N$155: D81.CKO, D82.CKI
- removed net N$156: D81.SDO, D82.SDI
- removed net N$157: D82.CKO, D83.CKI
- removed net N$158: D82.SDO, D83.SDI
- removed net N$159: D83.CKO, D84.CKI
- removed net N$160: D83.SDO, D84.SDI
- removed net N$161: D84.CKO, D85.CKI
- removed net N$162: D84.SDO, D85.SDI
- removed net N$163: D85.CKO, D86.CKI
- removed net N$164: D85.SDO, D86.SDI
- removed net N$165: D86.CKO, D87.CKI
- removed net N$166: D86.SDO, D87.SDI
- removed net N$167: D87.CKO, D88.CKI
- removed net N$168: D87.SDO, D88.SDI
- removed net N$169: D89.CKO, D90.CKI
- removed net N$170: D89.SDO, D90.SDI
- removed net N$171: D91.CKO, D92.CKI
- removed net N$172: D91.SDO, D92.SDI
- removed net N$173: D92.CKO, D93.CKI
- removed net N$174: D92.SDO, D93.SDI
- removed net N$175: D93.CKO, D94.CKI
- removed net N$176: D93.SDO, D94.SDI
- removed net N$177: D94.CKO, D95.CKI
- removed net N$178: D94.SDO, D95.SDI
- removed net N$179: D95.CKO, D96.CKI
- removed net N$180: D95.SDO, D96.SDI
- removed net N$181: D97.CKO, D98.CKI
- removed net N$182: D97.SDO, D98.SDI
- removed net N$183: D98.SDO, D99.SDI
- removed net N$184: D100.CKI, D99.CKO
- removed net N$185: D100.SDI, D99.SDO
- removed net N$186: D98.CKO, D99.CKI
- removed net N$187: D88.CKO, D89.CKI
- removed net N$188: D88.SDO, D89.SDI
- removed net N$189: D96.SDO, D97.SDI
- removed net N$190: D96.CKO, D97.CKI
- removed net N$191: D101.CKO, D102.CKI
- removed net N$192: D101.SDO, D102.SDI
- removed net N$193: D102.CKO, D103.CKI
- removed net N$194: D102.SDO, D103.SDI
- removed net N$195: D103.CKO, D104.CKI
- removed net N$196: D103.SDO, D104.SDI
- removed net N$197: D104.CKO, D105.CKI
- removed net N$198: D104.SDO, D105.SDI
- removed net N$199: D106.CKO, D107.CKI
- removed net N$2: D61.CKO, D71.CKI
- removed net N$200: D106.SDO, D107.SDI
- removed net N$201: D107.CKO, D108.CKI
- removed net N$202: D107.SDO, D108.SDI
- removed net N$203: D109.CKO, D110.CKI
- removed net N$204: D109.SDO, D110.SDI
- removed net N$205: D110.CKO, D111.CKI
- removed net N$206: D110.SDO, D111.SDI
- removed net N$207: D111.CKO, D112.CKI
- removed net N$208: D111.SDO, D112.SDI
- removed net N$209: D112.CKO, D113.CKI
- removed net N$210: D112.SDO, D113.SDI
- removed net N$211: D113.CKO, D114.CKI
- removed net N$212: D113.SDO, D114.SDI
- removed net N$213: D114.CKO, D115.CKI
- removed net N$214: D114.SDO, D115.SDI
- removed net N$215: D115.CKO, D116.CKI
- removed net N$216: D115.SDO, D116.SDI
- removed net N$217: D117.CKO, D118.CKI
- removed net N$218: D117.SDO, D118.SDI
- removed net N$219: D118.SDO, D119.SDI
- removed net N$220: D119.CKO, D120.CKI
- removed net N$221: D119.SDO, D120.SDI
- removed net N$222: D118.CKO, D119.CKI
- removed net N$223: D108.CKO, D109.CKI
- removed net N$224: D108.SDO, D109.SDI
- removed net N$225: D116.SDO, D117.SDI
- removed net N$226: D116.CKO, D117.CKI
- removed net N$227: D80.CKO, D81.CKI
- removed net N$228: D80.SDO, D81.SDI
- removed net N$229: D105.CKO, D106.CKI
- removed net N$230: D90.CKO, D91.CKI
- removed net N$231: D90.SDO, D91.SDI
- removed net N$232: D67.CKO, D68.CKI
- removed net N$233: D67.SDO, D68.SDI
- removed net N$234: D105.SDO, D106.SDI
- removed net N$235: D100.CKO, D101.CKI
- removed net N$236: D100.SDO, D101.SDI
- removed net N$237: D121.CKO, D131.CKI
- removed net N$238: D121.SDO, D131.SDI
- removed net N$239: D131.CKO, D132.CKI
- removed net N$240: D131.SDO, D132.SDI
- removed net N$241: D132.CKO, D133.CKI
- removed net N$242: D132.SDO, D133.SDI
- removed net N$243: D133.CKO, D134.CKI
- removed net N$244: D133.SDO, D134.SDI
- removed net N$245: D134.CKO, D135.CKI
- removed net N$246: D134.SDO, D135.SDI
- removed net N$247: D135.CKO, D136.CKI
- removed net N$248: D135.SDO, D136.SDI
- removed net N$249: D136.CKO, D137.CKI
- removed net N$250: D136.SDO, D137.SDI
- removed net N$251: D122.CKI, D138.CKO
- removed net N$252: D122.SDI, D138.SDO
- removed net N$253: D122.CKO, D123.CKI
- removed net N$254: D122.SDO, D123.SDI
- removed net N$255: D123.CKO, D124.CKI
- removed net N$256: D123.SDO, D124.SDI
- removed net N$257: D124.CKO, D125.CKI
- removed net N$258: D124.SDO, D125.SDI
- removed net N$259: D125.CKO, D126.CKI
- removed net N$260: D125.SDO, D126.SDI
- removed net N$261: D126.CKO, D127.CKI
- removed net N$262: D126.SDO, D127.SDI
- removed net N$263: D129.CKO, D130.CKI
- removed net N$264: D129.SDO, D130.SDI
- removed net N$265: D130.SDO, D139.SDI
- removed net N$266: D139.CKO, D140.CKI
- removed net N$267: D139.SDO, D140.SDI
- removed net N$268: D130.CKO, D139.CKI
- removed net N$269: D137.CKO, D138.CKI
- removed net N$270: D137.SDO, D138.SDI
- removed net N$271: D128.SDO, D129.SDI
- removed net N$272: D128.CKO, D129.CKI
- removed net N$273: D141.CKO, D142.CKI
- removed net N$274: D141.SDO, D142.SDI
- removed net N$275: D142.CKO, D143.CKI
- removed net N$276: D142.SDO, D143.SDI
- removed net N$277: D143.CKO, D144.CKI
- removed net N$278: D143.SDO, D144.SDI
- removed net N$279: D144.CKO, D145.CKI
- removed net N$280: D144.SDO, D145.SDI
- removed net N$281: D145.CKO, D146.CKI
- removed net N$282: D145.SDO, D146.SDI
- removed net N$283: D146.CKO, D147.CKI
- removed net N$284: D146.SDO, D147.SDI
- removed net N$285: D147.CKO, D148.CKI
- removed net N$286: D147.SDO, D148.SDI
- removed net N$287: D149.CKO, D150.CKI
- removed net N$288: D149.SDO, D150.SDI
- removed net N$289: D151.CKO, D152.CKI
- removed net N$290: D151.SDO, D152.SDI
- removed net N$291: D152.CKO, D153.CKI
- removed net N$292: D152.SDO, D153.SDI
- removed net N$293: D153.CKO, D154.CKI
- removed net N$294: D153.SDO, D154.SDI
- removed net N$295: D154.CKO, D155.CKI
- removed net N$296: D154.SDO, D155.SDI
- removed net N$297: D155.CKO, D156.CKI
- removed net N$298: D155.SDO, D156.SDI
- removed net N$299: D157.CKO, D158.CKI
- removed net N$3: D61.SDO, D71.SDI
- removed net N$300: D157.SDO, D158.SDI
- removed net N$301: D158.SDO, D159.SDI
- removed net N$302: D159.CKO, D160.CKI
- removed net N$303: D159.SDO, D160.SDI
- removed net N$304: D158.CKO, D159.CKI
- removed net N$305: D148.CKO, D149.CKI
- removed net N$306: D148.SDO, D149.SDI
- removed net N$307: D156.SDO, D157.SDI
- removed net N$308: D156.CKO, D157.CKI
- removed net N$309: D161.CKO, D162.CKI
- removed net N$310: D161.SDO, D162.SDI
- removed net N$311: D162.CKO, D163.CKI
- removed net N$312: D162.SDO, D163.SDI
- removed net N$313: D163.CKO, D164.CKI
- removed net N$314: D163.SDO, D164.SDI
- removed net N$315: D164.CKO, D165.CKI
- removed net N$316: D164.SDO, D165.SDI
- removed net N$317: D166.CKO, D167.CKI
- removed net N$318: D166.SDO, D167.SDI
- removed net N$319: D167.CKO, D168.CKI
- removed net N$320: D167.SDO, D168.SDI
- removed net N$321: D169.CKO, D170.CKI
- removed net N$322: D169.SDO, D170.SDI
- removed net N$323: D170.CKO, D171.CKI
- removed net N$324: D170.SDO, D171.SDI
- removed net N$325: D171.CKO, D172.CKI
- removed net N$326: D171.SDO, D172.SDI
- removed net N$327: D172.CKO, D173.CKI
- removed net N$328: D172.SDO, D173.SDI
- removed net N$329: D173.CKO, D174.CKI
- removed net N$330: D173.SDO, D174.SDI
- removed net N$331: D174.CKO, D175.CKI
- removed net N$332: D174.SDO, D175.SDI
- removed net N$333: D175.CKO, D176.CKI
- removed net N$334: D175.SDO, D176.SDI
- removed net N$335: D177.CKO, D178.CKI
- removed net N$336: D177.SDO, D178.SDI
- removed net N$337: D178.SDO, D179.SDI
- removed net N$338: D179.CKO, D180.CKI
- removed net N$339: D179.SDO, D180.SDI
- removed net N$340: D178.CKO, D179.CKI
- removed net N$341: D168.CKO, D169.CKI
- removed net N$342: D168.SDO, D169.SDI
- removed net N$343: D176.SDO, D177.SDI
- removed net N$344: D176.CKO, D177.CKI
- removed net N$345: D140.CKO, D141.CKI
- removed net N$346: D140.SDO, D141.SDI
- removed net N$347: D165.CKO, D166.CKI
- removed net N$348: D150.CKO, D151.CKI
- removed net N$349: D150.SDO, D151.SDI
- removed net N$350: D127.CKO, D128.CKI
- removed net N$351: D127.SDO, D128.SDI
- removed net N$352: D165.SDO, D166.SDI
- removed net N$353: D160.CKO, D161.CKI
- removed net N$354: D160.SDO, D161.SDI
- removed net N$355: D181.CKO, D191.CKI
- removed net N$356: D181.SDO, D191.SDI
- removed net N$357: D191.CKO, D192.CKI
- removed net N$358: D191.SDO, D192.SDI
- removed net N$359: D192.CKO, D193.CKI
- removed net N$360: D192.SDO, D193.SDI
- removed net N$361: D193.CKO, D194.CKI
- removed net N$362: D193.SDO, D194.SDI
- removed net N$363: D194.CKO, D195.CKI
- removed net N$364: D194.SDO, D195.SDI
- removed net N$365: D195.CKO, D196.CKI
- removed net N$366: D195.SDO, D196.SDI
- removed net N$367: D196.CKO, D197.CKI
- removed net N$368: D196.SDO, D197.SDI
- removed net N$369: D182.CKI, D198.CKO
- removed net N$370: D182.SDI, D198.SDO
- removed net N$371: D182.CKO, D183.CKI
- removed net N$372: D182.SDO, D183.SDI
- removed net N$373: D183.CKO, D184.CKI
- removed net N$374: D183.SDO, D184.SDI
- removed net N$375: D184.CKO, D185.CKI
- removed net N$376: D184.SDO, D185.SDI
- removed net N$377: D185.CKO, D186.CKI
- removed net N$378: D185.SDO, D186.SDI
- removed net N$379: D186.CKO, D187.CKI
- removed net N$380: D186.SDO, D187.SDI
- removed net N$381: D189.CKO, D190.CKI
- removed net N$382: D189.SDO, D190.SDI
- removed net N$383: D190.SDO, D199.SDI
- removed net N$384: D199.CKO, D200.CKI
- removed net N$385: D199.SDO, D200.SDI
- removed net N$386: D190.CKO, D199.CKI
- removed net N$387: D197.CKO, D198.CKI
- removed net N$388: D197.SDO, D198.SDI
- removed net N$389: D188.SDO, D189.SDI
- removed net N$390: D188.CKO, D189.CKI
- removed net N$391: D201.CKO, D202.CKI
- removed net N$392: D201.SDO, D202.SDI
- removed net N$393: D202.CKO, D203.CKI
- removed net N$394: D202.SDO, D203.SDI
- removed net N$395: D203.CKO, D204.CKI
- removed net N$396: D203.SDO, D204.SDI
- removed net N$397: D204.CKO, D205.CKI
- removed net N$398: D204.SDO, D205.SDI
- removed net N$399: D205.CKO, D206.CKI
- removed net N$400: D205.SDO, D206.SDI
- removed net N$401: D206.CKO, D207.CKI
- removed net N$402: D206.SDO, D207.SDI
- removed net N$403: D207.CKO, D208.CKI
- removed net N$404: D207.SDO, D208.SDI
- removed net N$405: D209.CKO, D210.CKI
- removed net N$406: D209.SDO, D210.SDI
- removed net N$407: D211.CKO, D212.CKI
- removed net N$408: D211.SDO, D212.SDI
- removed net N$409: D212.CKO, D213.CKI
- removed net N$410: D212.SDO, D213.SDI
- removed net N$411: D213.CKO, D214.CKI
- removed net N$412: D213.SDO, D214.SDI
- removed net N$413: D214.CKO, D215.CKI
- removed net N$414: D214.SDO, D215.SDI
- removed net N$415: D215.CKO, D216.CKI
- removed net N$416: D215.SDO, D216.SDI
- removed net N$417: D217.CKO, D218.CKI
- removed net N$418: D217.SDO, D218.SDI
- removed net N$419: D218.SDO, D219.SDI
- removed net N$420: D219.CKO, D220.CKI
- removed net N$421: D219.SDO, D220.SDI
- removed net N$422: D218.CKO, D219.CKI
- removed net N$423: D208.CKO, D209.CKI
- removed net N$424: D208.SDO, D209.SDI
- removed net N$425: D216.SDO, D217.SDI
- removed net N$426: D216.CKO, D217.CKI
- removed net N$427: D221.CKO, D222.CKI
- removed net N$428: D221.SDO, D222.SDI
- removed net N$429: D222.CKO, D223.CKI
- removed net N$430: D222.SDO, D223.SDI
- removed net N$431: D223.CKO, D224.CKI
- removed net N$432: D223.SDO, D224.SDI
- removed net N$433: D224.CKO, D225.CKI
- removed net N$434: D224.SDO, D225.SDI
- removed net N$435: D226.CKO, D227.CKI
- removed net N$436: D226.SDO, D227.SDI
- removed net N$437: D227.CKO, D228.CKI
- removed net N$438: D227.SDO, D228.SDI
- removed net N$439: D229.CKO, D230.CKI
- removed net N$440: D229.SDO, D230.SDI
- removed net N$441: D230.CKO, D231.CKI
- removed net N$442: D230.SDO, D231.SDI
- removed net N$443: D231.CKO, D232.CKI
- removed net N$444: D231.SDO, D232.SDI
- removed net N$445: D232.CKO, D233.CKI
- removed net N$446: D232.SDO, D233.SDI
- removed net N$447: D233.CKO, D234.CKI
- removed net N$448: D233.SDO, D234.SDI
- removed net N$449: D234.CKO, D235.CKI
- removed net N$450: D234.SDO, D235.SDI
- removed net N$451: D235.CKO, D236.CKI
- removed net N$452: D235.SDO, D236.SDI
- removed net N$453: D237.CKO, D238.CKI
- removed net N$454: D237.SDO, D238.SDI
- removed net N$455: D238.SDO, D239.SDI
- removed net N$456: D239.CKO, D240.CKI
- removed net N$457: D239.SDO, D240.SDI
- removed net N$458: D238.CKO, D239.CKI
- removed net N$459: D228.CKO, D229.CKI
- removed net N$460: D228.SDO, D229.SDI
- removed net N$461: D236.SDO, D237.SDI
- removed net N$462: D236.CKO, D237.CKI
- removed net N$463: D200.CKO, D201.CKI
- removed net N$464: D200.SDO, D201.SDI
- removed net N$465: D225.CKO, D226.CKI
- removed net N$466: D210.CKO, D211.CKI
- removed net N$467: D210.SDO, D211.SDI
- removed net N$468: D187.CKO, D188.CKI
- removed net N$469: D187.SDO, D188.SDI
- removed net N$470: D225.SDO, D226.SDI
- removed net N$471: D220.CKO, D221.CKI
- removed net N$472: D220.SDO, D221.SDI
- removed net N$473: D241.CKO, D251.CKI
- removed net N$474: D241.SDO, D251.SDI
- removed net N$475: D251.CKO, D252.CKI
- removed net N$476: D251.SDO, D252.SDI
- removed net N$477: D252.CKO, D253.CKI
- removed net N$478: D252.SDO, D253.SDI
- removed net N$479: D253.CKO, D254.CKI
- removed net N$480: D253.SDO, D254.SDI
- removed net N$481: D254.CKO, D255.CKI
- removed net N$482: D254.SDO, D255.SDI
- removed net N$483: D255.CKO, D256.CKI
- removed net N$484: D255.SDO, D256.SDI
- removed net N$485: D256.CKO, D257.CKI
- removed net N$486: D256.SDO, D257.SDI
- removed net N$487: D242.CKI, D258.CKO
- removed net N$488: D242.SDI, D258.SDO
- removed net N$489: D242.CKO, D243.CKI
- removed net N$490: D242.SDO, D243.SDI
- removed net N$491: D243.CKO, D244.CKI
- removed net N$492: D243.SDO, D244.SDI
- removed net N$493: D244.CKO, D245.CKI
- removed net N$494: D244.SDO, D245.SDI
- removed net N$495: D245.CKO, D246.CKI
- removed net N$496: D245.SDO, D246.SDI
- removed net N$497: D246.CKO, D247.CKI
- removed net N$498: D246.SDO, D247.SDI
- removed net N$499: D249.CKO, D250.CKI
- removed net N$500: D249.SDO, D250.SDI
- removed net N$501: D250.SDO, D259.SDI
- removed net N$502: D259.CKO, D260.CKI
- removed net N$503: D259.SDO, D260.SDI
- removed net N$504: D250.CKO, D259.CKI
- removed net N$505: D257.CKO, D258.CKI
- removed net N$506: D257.SDO, D258.SDI
- removed net N$507: D248.SDO, D249.SDI
- removed net N$508: D248.CKO, D249.CKI
- removed net N$509: D261.CKO, D262.CKI
- removed net N$510: D261.SDO, D262.SDI
- removed net N$511: D262.CKO, D263.CKI
- removed net N$512: D262.SDO, D263.SDI
- removed net N$513: D263.CKO, D264.CKI
- removed net N$514: D263.SDO, D264.SDI
- removed net N$515: D264.CKO, D265.CKI
- removed net N$516: D264.SDO, D265.SDI
- removed net N$517: D265.CKO, D266.CKI
- removed net N$518: D265.SDO, D266.SDI
- removed net N$519: D266.CKO, D267.CKI
- removed net N$520: D266.SDO, D267.SDI
- removed net N$521: D267.CKO, D268.CKI
- removed net N$522: D267.SDO, D268.SDI
- removed net N$523: D269.CKO, D270.CKI
- removed net N$524: D269.SDO, D270.SDI
- removed net N$525: D271.CKO, D272.CKI
- removed net N$526: D271.SDO, D272.SDI
- removed net N$527: D272.CKO, D273.CKI
- removed net N$528: D272.SDO, D273.SDI
- removed net N$529: D273.CKO, D274.CKI
- removed net N$530: D273.SDO, D274.SDI
- removed net N$531: D274.CKO, D275.CKI
- removed net N$532: D274.SDO, D275.SDI
- removed net N$533: D275.CKO, D276.CKI
- removed net N$534: D275.SDO, D276.SDI
- removed net N$535: D277.CKO, D278.CKI
- removed net N$536: D277.SDO, D278.SDI
- removed net N$537: D278.SDO, D279.SDI
- removed net N$538: D279.CKO, D280.CKI
- removed net N$539: D279.SDO, D280.SDI
- removed net N$540: D278.CKO, D279.CKI
- removed net N$541: D268.CKO, D269.CKI
- removed net N$542: D268.SDO, D269.SDI
- removed net N$543: D276.SDO, D277.SDI
- removed net N$544: D276.CKO, D277.CKI
- removed net N$545: D281.CKO, D282.CKI
- removed net N$546: D281.SDO, D282.SDI
- removed net N$547: D282.CKO, D283.CKI
- removed net N$548: D282.SDO, D283.SDI
- removed net N$549: D283.CKO, D284.CKI
- removed net N$550: D283.SDO, D284.SDI
- removed net N$551: D284.CKO, D285.CKI
- removed net N$552: D284.SDO, D285.SDI
- removed net N$553: D286.CKO, D287.CKI
- removed net N$554: D286.SDO, D287.SDI
- removed net N$555: D287.CKO, D288.CKI
- removed net N$556: D287.SDO, D288.SDI
- removed net N$557: D289.CKO, D290.CKI
- removed net N$558: D289.SDO, D290.SDI
- removed net N$559: D290.CKO, D291.CKI
- removed net N$560: D290.SDO, D291.SDI
- removed net N$561: D291.CKO, D292.CKI
- removed net N$562: D291.SDO, D292.SDI
- removed net N$563: D292.CKO, D293.CKI
- removed net N$564: D292.SDO, D293.SDI
- removed net N$565: D293.CKO, D294.CKI
- removed net N$566: D293.SDO, D294.SDI
- removed net N$567: D294.CKO, D295.CKI
- removed net N$568: D294.SDO, D295.SDI
- removed net N$569: D295.CKO, D296.CKI
- removed net N$570: D295.SDO, D296.SDI
- removed net N$571: D297.CKO, D298.CKI
- removed net N$572: D297.SDO, D298.SDI
- removed net N$573: D298.SDO, D299.SDI
- removed net N$574: D299.CKO, D300.CKI
- removed net N$575: D299.SDO, D300.SDI
- removed net N$576: D298.CKO, D299.CKI
- removed net N$577: D288.CKO, D289.CKI
- removed net N$578: D288.SDO, D289.SDI
- removed net N$579: D296.SDO, D297.SDI
- removed net N$580: D296.CKO, D297.CKI
- removed net N$581: D260.CKO, D261.CKI
- removed net N$582: D260.SDO, D261.SDI
- removed net N$583: D285.CKO, D286.CKI
- removed net N$584: D270.CKO, D271.CKI
- removed net N$585: D270.SDO, D271.SDI
- removed net N$586: D247.CKO, D248.CKI
- removed net N$587: D247.SDO, D248.SDI
- removed net N$588: D285.SDO, D286.SDI
- removed net N$589: D280.CKO, D281.CKI
- removed net N$590: D280.SDO, D281.SDI
- removed net N$591: D301.CKO, D311.CKI
- removed net N$592: D301.SDO, D311.SDI
- removed net N$593: D311.CKO, D312.CKI
- removed net N$594: D311.SDO, D312.SDI
- removed net N$595: D312.CKO, D313.CKI
- removed net N$596: D312.SDO, D313.SDI
- removed net N$597: D313.CKO, D314.CKI
- removed net N$598: D313.SDO, D314.SDI
- removed net N$599: D314.CKO, D315.CKI
- removed net N$600: D314.SDO, D315.SDI
- removed net N$601: D315.CKO, D316.CKI
- removed net N$602: D315.SDO, D316.SDI
- removed net N$603: D316.CKO, D317.CKI
- removed net N$604: D316.SDO, D317.SDI
- removed net N$605: D302.CKI, D318.CKO
- removed net N$606: D302.SDI, D318.SDO
- removed net N$607: D302.CKO, D303.CKI
- removed net N$608: D302.SDO, D303.SDI
- removed net N$609: D303.CKO, D304.CKI
- removed net N$610: D303.SDO, D304.SDI
- removed net N$611: D304.CKO, D305.CKI
- removed net N$612: D304.SDO, D305.SDI
- removed net N$613: D305.CKO, D306.CKI
- removed net N$614: D305.SDO, D306.SDI
- removed net N$615: D306.CKO, D307.CKI
- removed net N$616: D306.SDO, D307.SDI
- removed net N$617: D309.CKO, D310.CKI
- removed net N$618: D309.SDO, D310.SDI
- removed net N$619: D310.SDO, D319.SDI
- removed net N$620: D319.CKO, D320.CKI
- removed net N$621: D319.SDO, D320.SDI
- removed net N$622: D310.CKO, D319.CKI
- removed net N$623: D317.CKO, D318.CKI
- removed net N$624: D317.SDO, D318.SDI
- removed net N$625: D308.SDO, D309.SDI
- removed net N$626: D308.CKO, D309.CKI
- removed net N$627: D321.CKO, D322.CKI
- removed net N$628: D321.SDO, D322.SDI
- removed net N$629: D322.CKO, D323.CKI
- removed net N$630: D322.SDO, D323.SDI
- removed net N$631: D323.CKO, D324.CKI
- removed net N$632: D323.SDO, D324.SDI
- removed net N$633: D324.CKO, D325.CKI
- removed net N$634: D324.SDO, D325.SDI
- removed net N$635: D325.CKO, D326.CKI
- removed net N$636: D325.SDO, D326.SDI
- removed net N$637: D326.CKO, D327.CKI
- removed net N$638: D326.SDO, D327.SDI
- removed net N$639: D327.CKO, D328.CKI
- removed net N$640: D327.SDO, D328.SDI
- removed net N$641: D329.CKO, D330.CKI
- removed net N$642: D329.SDO, D330.SDI
- removed net N$643: D331.CKO, D332.CKI
- removed net N$644: D331.SDO, D332.SDI
- removed net N$645: D332.CKO, D333.CKI
- removed net N$646: D332.SDO, D333.SDI
- removed net N$647: D333.CKO, D334.CKI
- removed net N$648: D333.SDO, D334.SDI
- removed net N$649: D334.CKO, D335.CKI
- removed net N$650: D334.SDO, D335.SDI
- removed net N$651: D335.CKO, D336.CKI
- removed net N$652: D335.SDO, D336.SDI
- removed net N$653: D337.CKO, D338.CKI
- removed net N$654: D337.SDO, D338.SDI
- removed net N$655: D338.SDO, D339.SDI
- removed net N$656: D339.CKO, D340.CKI
- removed net N$657: D339.SDO, D340.SDI
- removed net N$658: D338.CKO, D339.CKI
- removed net N$659: D328.CKO, D329.CKI
- removed net N$660: D328.SDO, D329.SDI
- removed net N$661: D336.SDO, D337.SDI
- removed net N$662: D336.CKO, D337.CKI
- removed net N$663: D341.CKO, D342.CKI
- removed net N$664: D341.SDO, D342.SDI
- removed net N$665: D342.CKO, D343.CKI
- removed net N$666: D342.SDO, D343.SDI
- removed net N$667: D343.CKO, D344.CKI
- removed net N$668: D343.SDO, D344.SDI
- removed net N$669: D344.CKO, D345.CKI
- removed net N$670: D344.SDO, D345.SDI
- removed net N$671: D346.CKO, D347.CKI
- removed net N$672: D346.SDO, D347.SDI
- removed net N$673: D347.CKO, D348.CKI
- removed net N$674: D347.SDO, D348.SDI
- removed net N$675: D349.CKO, D350.CKI
- removed net N$676: D349.SDO, D350.SDI
- removed net N$677: D350.CKO, D351.CKI
- removed net N$678: D350.SDO, D351.SDI
- removed net N$679: D351.CKO, D352.CKI
- removed net N$680: D351.SDO, D352.SDI
- removed net N$681: D352.CKO, D353.CKI
- removed net N$682: D352.SDO, D353.SDI
- removed net N$683: D353.CKO, D354.CKI
- removed net N$684: D353.SDO, D354.SDI
- removed net N$685: D354.CKO, D355.CKI
- removed net N$686: D354.SDO, D355.SDI
- removed net N$687: D355.CKO, D356.CKI
- removed net N$688: D355.SDO, D356.SDI
- removed net N$689: D357.CKO, D358.CKI
- removed net N$690: D357.SDO, D358.SDI
- removed net N$691: D358.SDO, D359.SDI
- removed net N$692: D359.CKO, D360.CKI
- removed net N$693: D359.SDO, D360.SDI
- removed net N$694: D358.CKO, D359.CKI
- removed net N$695: D348.CKO, D349.CKI
- removed net N$696: D348.SDO, D349.SDI
- removed net N$697: D356.SDO, D357.SDI
- removed net N$698: D356.CKO, D357.CKI
- removed net N$699: D320.CKO, D321.CKI
- removed net N$700: D320.SDO, D321.SDI
- removed net N$701: D345.CKO, D346.CKI
- removed net N$702: D330.CKO, D331.CKI
- removed net N$703: D330.SDO, D331.SDI
- removed net N$704: D307.CKO, D308.CKI
- removed net N$705: D307.SDO, D308.SDI
- removed net N$706: D345.SDO, D346.SDI
- removed net N$707: D340.CKO, D341.CKI
- removed net N$708: D340.SDO, D341.SDI
- removed net N$92: D71.CKO, D72.CKI
- removed net N$93: D71.SDO, D72.SDI
Routing:
- net DO4: track 5.06 -> 0.00 mm, vias 1 -> 0
- net DO2: track 5.06 -> 0.00 mm, vias 1 -> 0
- net DO5: track 5.06 -> 0.00 mm, vias 1 -> 0
- net DO3: track 5.06 -> 0.00 mm, vias 1 -> 0
- net DO1: track 5.06 -> 0.00 mm, vias 1 -> 0
- net 5V3: track 4.53 -> 0.00 mm, vias 2 -> 0
- net 5V5: track 4.53 -> 0.00 mm, vias 2 -> 0
- net 5V1: track 4.53 -> 0.00 mm, vias 2 -> 0
- net 5V2: track 4.53 -> 0.00 mm, vias 2 -> 0
- net 5V4: track 4.53 -> 0.00 mm, vias 2 -> 0
- net DI4: track 4.11 -> 0.00 mm, vias 1 -> 0
- net DI2: track 4.11 -> 0.00 mm, vias 1 -> 0
- net DI5: track 4.11 -> 0.00 mm, vias 1 -> 0
- net DI3: track 4.11 -> 0.00 mm, vias 1 -> 0
- net DI1: track 4.11 -> 0.00 mm, vias 1 -> 0
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- removed copper zone on layer 1, net 5V1
- removed copper zone on layer 1, net 5V2
- removed copper zone on layer 1, net 5V3
- removed copper zone on layer 1, net 5V4
- removed copper zone on layer 1, net 5V5
- removed copper zone on layer 1, net GND1
- removed copper zone on layer 16, net GND1
- removed copper zone on layer 1, net GND2
- removed copper zone on layer 16, net GND2
- removed copper zone on layer 1, net GND3
- removed copper zone on layer 16, net GND3
- removed copper zone on layer 1, net GND4
- removed copper zone on layer 16, net GND4
- removed copper zone on layer 1, net GND5
- removed copper zone on layer 16, net GND5
Other:
- board size 166.6 x 243.3 mm -> 76.2 x 76.2 mm
- board text added: "Andy England"
- board text added: "Black PCB"
- board text removed: "Route OUT"
- board text removed: "Route Out"
