File: Hardware/LuMini_3Inch.sch (EAGLE design)
At the start: 79 parts, among them J1 DOUBLE_LED_PAD, J2 DOUBLE_LED_PAD, J3 DOUBLE_LED_PAD

Commit message: fixing library issue
Parts:
- J1, J2, J3: value DOUBLE_LED_PAD -> SOLDER_PAD_2; device Andy:DOUBLE_LED_PAD -> SparkFun-Connectors:SOLDER_PAD_2
Other:
- moved on the sheet: H1, H2, H3, H5, H6, H7
Changed lines of the file:
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@@
 <part name="SUPPLY21" library="SparkFun-PowerSymbols" deviceset="5V" device=""/>
 <part name="GND21" library="SparkFun-PowerSymbols" deviceset="GND" device=""/>
-<part name="J1" library="Andy" deviceset="DOUBLE_LED_PAD" device=""/>
-<part name="J2" library="Andy" deviceset="DOUBLE_LED_PAD" device=""/>
+<part name="J1" library="SparkFun-Connectors" deviceset="SOLDER_PAD_2" device=""/>
+<part name="J2" library="SparkFun-Connectors" deviceset="SOLDER_PAD_2" device=""/>
 <part name="D21" library="SparkFun-LED" deviceset="APA102" device="2020"/>
 <part name="SUPPLY22" library="SparkFun-PowerSymbols" deviceset="5V" device=""/>
@@
 <part name="SUPPLY61" library="SparkFun-PowerSymbols" deviceset="5V" device=""/>
 <part name="GND61" library="SparkFun-PowerSymbols" deviceset="GND" device=""/>
-<part name="J3" library="Andy" deviceset="DOUBLE_LED_PAD" device=""/>
+<part name="J3" library="SparkFun-Connectors" deviceset="SOLDER_PAD_2" device=""/>
 <part name="FRAME1" library="SparkFun-Aesthetics" deviceset="FRAME-LEDGER" device=""/>
 <part name="H1" library="SparkFun-Hardware" deviceset="STANDOFF_ELECTRICAL" device="-NOTHERMALS" value="STANDOFF_ELECTRICAL-NOTHERMALS"/>
@@
 <plain>
 <text x="200.66" y="264.16" size="3.81" layer="97" font="vector">LED's</text>
-<text x="218.44" y="111.76" size="3.81" layer="97" font="vector">Grounding Standoffs</text>
+<text x="218.44" y="114.3" size="3.81" layer="97" font="vector">Grounding Standoffs</text>
 <wire x1="0" y1="144.78" x2="149.86" y2="144.78" width="0.2032" layer="97" style="longdash"/>
 <text x="348.742" y="11.176" size="2.54" layer="94" font="vector">Andy England</text>
@@
 <instance part="FRAME1" gate="G$1" x="0" y="0"/>
 <instance part="FRAME1" gate="G$2" x="330.2" y="0"/>
-<instance part="H1" gate="G$1" x="248.92" y="99.06" rot="R180"/>
-<instance part="H2" gate="G$1" x="248.92" y="83.82" rot="R180"/>
-<instance part="H3" gate="G$1" x="248.92" y="68.58" rot="R180"/>
+<instance part="H1" gate="G$1" x="248.92" y="104.14" rot="R180"/>
+<instance part="H2" gate="G$1" x="248.92" y="88.9" rot="R180"/>
+<instance part="H3" gate="G$1" x="248.92" y="71.12" rot="R180"/>
 <instance part="H4" gate="G$1" x="248.92" y="53.34" rot="R180"/>
 <instance part="GND17" gate="1" x="238.76" y="40.64"/>
@@
 <instance part="LOGO1" gate="G$1" x="411.48" y="45.72"/>
 <instance part="LOGO2" gate="G$1" x="335.28" y="38.1"/>
-<instance part="H5" gate="G$1" x="228.6" y="99.06"/>
-<instance part="H6" gate="G$1" x="228.6" y="81.28"/>
-<instance part="H7" gate="G$1" x="228.6" y="66.04"/>
+<instance part="H5" gate="G$1" x="228.6" y="104.14"/>
+<instance part="H6" gate="G$1" x="228.6" y="86.36"/>
+<instance part="H7" gate="G$1" x="228.6" y="68.58"/>
 <instance part="H8" gate="G$1" x="228.6" y="50.8"/>
 <instance part="FD1" gate="G$1" x="414.02" y="20.32"/>
@@
 <segment>
 <pinref part="H1" gate="G$1" pin="P$1"/>
-<wire x1="241.3" y1="99.06" x2="238.76" y2="99.06" width="0.1524" layer="91"/>
+<wire x1="241.3" y1="104.14" x2="238.76" y2="104.14" width="0.1524" layer="91"/>
 <pinref part="GND17" gate="1" pin="GND"/>
-<wire x1="238.76" y1="99.06" x2="238.76" y2="83.82" width="0.1524" layer="91"/>
+<wire x1="238.76" y1="104.14" x2="238.76" y2="88.9" width="0.1524" layer="91"/>
 <pinref part="H4" gate="G$1" pin="P$1"/>
-<wire x1="238.76" y1="83.82" x2="238.76" y2="81.28" width="0.1524" layer="91"/>
-<wire x1="238.76" y1="81.28" x2="238.76" y2="68.58" width="0.1524" layer="91"/>
-<wire x1="238.76" y1="68.58" x2="238.76" y2="66.04" width="0.1524" layer="91"/>
-<wire x1="238.76" y1="66.04" x2="238.76" y2="53.34" width="0.1524" layer="91"/>
+<wire x1="238.76" y1="88.9" x2="238.76" y2="86.36" width="0.1524" layer="91"/>
+<wire x1="238.76" y1="86.36" x2="238.76" y2="71.12" width="0.1524" layer="91"/>
+<wire x1="238.76" y1="71.12" x2="238.76" y2="68.58" width="0.1524" layer="91"/>
+<wire x1="238.76" y1="68.58" x2="238.76" y2="53.34" width="0.1524" layer="91"/>
 <wire x1="238.76" y1="53.34" x2="238.76" y2="50.8" width="0.1524" layer="91"/>
 <wire x1="238.76" y1="50.8" x2="238.76" y2="43.18" width="0.1524" layer="91"/>
@@
 <junction x="238.76" y="53.34"/>
 <pinref part="H3" gate="G$1" pin="P$1"/>
-<wire x1="241.3" y1="68.58" x2="238.76" y2="68.58" width="0.1524" layer="91"/>
+<wire x1="241.3" y1="71.12" x2="238.76" y2="71.12" width="0.1524" layer="91"/>
+<junction x="238.76" y="71.12"/>
+<pinref part="H2" gate="G$1" pin="P$1"/>
+<wire x1="241.3" y1="88.9" x2="238.76" y2="88.9" width="0.1524" layer="91"/>
+<junction x="238.76" y="88.9"/>
+<pinref part="H5" gate="G$1" pin="P$1"/>
+<wire x1="238.76" y1="104.14" x2="236.22" y2="104.14" width="0.1524" layer="91"/>
+<junction x="238.76" y="104.14"/>
+<pinref part="H6" gate="G$1" pin="P$1"/>
+<wire x1="236.22" y1="86.36" x2="238.76" y2="86.36" width="0.1524" layer="91"/>
+<junction x="238.76" y="86.36"/>
+<pinref part="H7" gate="G$1" pin="P$1"/>
+<wire x1="238.76" y1="68.58" x2="236.22" y2="68.58" width="0.1524" layer="91"/>
 <junction x="238.76" y="68.58"/>
-<pinref part="H2" gate="G$1" pin="P$1"/>
-<wire x1="241.3" y1="83.82" x2="238.76" y2="83.82" width="0.1524" layer="91"/>
-<junction x="238.76" y="83.82"/>
-<pinref part="H5" gate="G$1" pin="P$1"/>
-<wire x1="238.76" y1="99.06" x2="236.22" y2="99.06" width="0.1524" layer="91"/>
-<junction x="238.76" y="99.06"/>
-<pinref part="H6" gate="G$1" pin="P$1"/>
-<wire x1="236.22" y1="81.28" x2="238.76" y2="81.28" width="0.1524" layer="91"/>
-<junction x="238.76" y="81.28"/>
-<pinref part="H7" gate="G$1" pin="P$1"/>
-<wire x1="238.76" y1="66.04" x2="236.22" y2="66.04" width="0.1524" layer="91"/>
-<junction x="238.76" y="66.04"/>
 <pinref part="H8" gate="G$1" pin="P$1"/>
 <wire x1="236.22" y1="50.8" x2="238.76" y2="50.8" width="0.1524" layer="91"/>

Commit message: updating to proper 6-pin footprint
Parts:
- D1, D10, D11, D12, D13, D14, D15, D16, D17, D18, D19, D2, D20, D21, D22, D23, D24, D25, D26, D27, D28, D29, D3, D30, D31, D32, D33, D34, D35, D36, D37, D38, D39, D4, D40, D41, D42, D43, D44, D45, D46, D47, D48, D49, D5, D50, D51, D52, D53, D54, D55, D56, D57, D58, D59, D6, D60, D7, D8, D9: value APA1022020 -> APA102-2020; device SparkFun-LED:APA1022020 -> SparkFun-LED:APA102-2020

Commit message: version number change
Other:
- note added: "v10"
- note removed: "v03"
Changed lines of the file:
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@@
 <wire x1="0" y1="144.78" x2="149.86" y2="144.78" width="0.2032" layer="97" style="longdash"/>
 <text x="348.742" y="11.176" size="2.54" layer="94" font="vector">Andy England</text>
-<text x="419.1" y="7.62" size="2.54" layer="94" font="vector">v03</text>
+<text x="419.1" y="7.62" size="2.54" layer="94" font="vector">v10</text>
 <text x="200.66" y="261.62" size="1.778" layer="97" font="vector">Vin: 3.0V-5.5V</text>
 <wire x1="149.86" y1="144.78" x2="330.2" y2="144.78" width="0.2032" layer="97" style="longdash"/>
